File: pcb/rgb-v0.2/master-pcb.sch (KiCad schematic (older format))
At the start: 35 parts, among them IC1 5V_REG, IC2 MC_33003A/34063A, IC3 ATMEGA328P_TQFP, IC4 MAX3232, J1 SERIAL_POWER_OUT_L, J2 SERIAL_POWER_OUT_R, P1 AVR_ISP, Y1 16MHz

Commit message: working on footprint
Parts:
- removed R6: 10k_arr, ~, symbol R-ARRAY_X8-BUSSED
- added C15: 100uF, ~, symbol C
- added L2: 1uH, ~, symbol L
- added R10, R11, R12, R13, R6, R7, R8, R9: 10k, ~, symbol R
- C7: value C -> 470pF
- L1: value 500H -> 220uH
- R4: value R_1 -> 1k
- R5: value R_2 -> 5.6k
Connections:
- net ADDR_0: now also R6.2
- net ADDR_1: now also R7.2
- net ADDR_2: now also R8.2
- net ADDR_3: now also R9.2
- net ADDR_4: now also R10.2
- net ADDR_5: now also R11.2
- net ADDR_6: now also R12.2
- net ADDR_7: now also R13.2
- net GND: now also C15.1, R10.1, R11.1, R12.1, R13.1, R6.1, R7.1, R8.1, R9.1
- net V_REG: now also C15.2, L2.2; no longer C8.2, L1.1, R5.2
- new net: C8.2, L1.1, L2.1, R5.2

Commit message: still modifying
Parts:
- removed C4: 100uF, ~, symbol C
- removed R10, R11, R12, R13, R6, R7, R8, R9: 10k, ~, symbol R
- removed S2: ADDRESS, ~, symbol SPST_X8
- added C4: 100uF, ~, symbol C_POL
Connections:
- net GND: now also C4.2
- net V_BUS: now also C4.1
- net ADDR_0: no longer names the net of IC3.23 (PC0(ADC0/PCINT8))
- net ADDR_1: no longer names the net of IC3.24 (PC1(ADC1/PCINT9))
- net ADDR_2: no longer names the net of IC3.25 (PC2(ADC2/PCINT10))
- net ADDR_3: no longer names the net of IC3.26 (PC3(ADC3/PCINT11))
- net ADDR_4: no longer names the net of IC3.27 (PC4(ADC4/SDA/PCINT12))
- net ADDR_5: no longer names the net of IC3.28 (PC5(ADC5/SCL/PCINT13))
- net ADDR_6: no longer names the net of IC3.10 (PD6(PCINT22/OC0A/AIN0))
- net ADDR_7: no longer names the net of IC3.11 (PD7(PCINT23/AIN1))
- no-connect marks 13 -> 21
Other:
- note removed: "Address"
- moved on the sheet: C14, C15, C5, C6, C7, C8, D1, F1, IC1, IC2, L1, L2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
